File: test/test.sch (KiCad schematic (older format))
At the start: 3 parts, among them U1 AP2112K-3.3, U2 ATmega32U4-AU

Commit message: update
Parts:
- removed U1: AP2112K-3.3, Package_TO_SOT_SMD:SOT-23-5, symbol Regulator_Linear:AP2112K-3.3
- removed U2: ATmega32U4-AU, Package_QFP:TQFP-44_10x10mm_P0.8mm, symbol MCU_Microchip_ATmega:ATmega32U4-AU
- added A1: Arduino_Nano_v2.x, Module:Arduino_Nano, symbol MCU_Module:Arduino_Nano_v2.x
- added D1: LED, LED_SMD:LED_1206_3216Metric, symbol Device:LED
Connections:
- net labels added: +3V3, +5V, GND
- wire segments 0 -> 10
- no-connect marks 0 -> 25
Changed lines of the file:
@@
 encoding utf-8
 Sheet 1 1
-Title ""
-Date ""
-Rev ""
+Title "test"
+Date "2020-08-06"
+Rev "v2.0"
 Comp ""
 Comment1 ""
@@
 $EndDescr
 $Comp
-L Device:R R1
-U 1 1 5EE13BA3
-P 5000 2500
-F 0 "R1" H 5100 2550 50  0000 L CNN
-F 1 "R" H 5100 2500 50  0000 L CNN
-F 2 "Resistor_SMD:R_1206_3216Metric" V 4930 2500 50  0001 C CNN
-F 3 "~" H 5000 2500 50  0001 C CNN
-	1    5000 2500
+L MCU_Module:Arduino_Nano_v2.x A1
+U 1 1 5F2BC279
+P 7500 3400
+F 0 "A1" H 7150 4375 50  0000 C CNN
+F 1 "Arduino_Nano_v2.x" H 8075 2425 50  0000 C CNN
+F 2 "Module:Arduino_Nano" H 7500 3400 50  0001 C CIN
+F 3 "https://www.arduino.cc/en/uploads/Main/ArduinoNanoManual23.pdf" H 7500 3400 50  0001 C CNN
+	1    7500 3400
 	1    0    0    -1
 $EndComp
 $Comp
-L MCU_Microchip_ATmega:ATmega32U4-AU U2
-U 1 1 5EF38BC6
-P 8500 3250
-F 0 "U2" H 8500 1325 50  0000 C CNN
-F 1 "ATmega32U4-AU" H 8500 1225 50  0000 C CNN
-F 2 "Package_QFP:TQFP-44_10x10mm_P0.8mm" H 8500 3250 50  0001 C CIN
-F 3 "http://ww1.microchip.com/downloads/en/DeviceDoc/Atmel-7766-8-bit-AVR-ATmega16U4-32U4_Datasheet.pdf" H 8500 3250 50  0001 C CNN
-	1    8500 3250
+L power:GND #PWR0101
+U 1 1 5F2BF0D1
+P 7500 4650
+F 0 "#PWR0101" H 7500 4400 50  0001 C CNN
+F 1 "GND" H 7550 4450 50  0000 C CNN
+F 2 "" H 7500 4650 50  0001 C CNN
+F 3 "" H 7500 4650 50  0001 C CNN
+	1    7500 4650
+	1    0    0    -1
+$EndComp
+Wire Wire Line
+	7500 4650 7500 4525
+Wire Wire Line
+	7600 4400 7600 4525
+Wire Wire Line
+	7600 4525 7500 4525
+Connection ~ 7500 4525
+Wire Wire Line
+	7500 4525 7500 4400
+NoConn ~ 7400 2400
+NoConn ~ 8000 4100
+NoConn ~ 8000 4000
+NoConn ~ 8000 3900
+NoConn ~ 8000 3800
+NoConn ~ 8000 3700
+NoConn ~ 8000 3600
+NoConn ~ 8000 3500
+NoConn ~ 8000 3400
+NoConn ~ 8000 3200
+NoConn ~ 8000 2900
+NoConn ~ 8000 2800
+NoConn ~ 7000 3700
+NoConn ~ 7000 3600
+NoConn ~ 7000 3500
+NoConn ~ 7000 3400
+NoConn ~ 7000 3300
+NoConn ~ 7000 3200
+NoConn ~ 7000 3100
+NoConn ~ 7000 3000
+NoConn ~ 7000 2900
+NoConn ~ 7000 2800
+NoConn ~ 7000 4100
+NoConn ~ 7000 4000
+NoConn ~ 7000 3900
+$Comp
+L Device:LED D1
+U 1 1 5F2C4A16
+P 6000 3800
+F 0 "D1" H 6000 4050 50  0000 C CNN
+F 1 "LED" H 6000 3950 50  0000 C CNN
+F 2 "LED_SMD:LED_1206_3216Metric" H 6000 3800 50  0001 C CNN
+F 3 "~" H 6000 3800 50  0001 C CNN
+	1    6000 3800
 	1    0    0    -1
 $EndComp
 $Comp
-L Regulator_Linear:AP2112K-3.3 U1
-U 1 1 5EF3B71C
-P 2750 2500
-F 0 "U1" H 2750 2900 50  0000 C CNN
-F 1 "AP2112K-3.3" H 2750 2800 50  0000 C CNN
-F 2 "Package_TO_SOT_SMD:SOT-23-5" H 2750 2825 50  0001 C CNN
-F 3 "https://www.diodes.com/assets/Datasheets/AP2112.pdf" H 2750 2600 50  0001 C CNN
-	1    2750 2500
+L Device:R R1
+U 1 1 5F2C57D7
+P 5500 4125
+F 0 "R1" H 5600 4200 50  0000 L CNN
+F 1 "R" H 5600 4100 50  0000 L CNN
+F 2 "Resistor_SMD:R_1206_3216Metric" V 5430 4125 50  0001 C CNN
+F 3 "~" H 5500 4125 50  0001 C CNN
+	1    5500 4125
 	1    0    0    -1
 $EndComp
+Wire Wire Line
+	7000 3800 6150 3800
+$Comp
+L power:GND #PWR0104
+U 1 1 5F2C5E83
+P 5500 4525
+F 0 "#PWR0104" H 5500 4275 50  0001 C CNN
+F 1 "GND" H 5500 4375 50  0000 C CNN
+F 2 "" H 5500 4525 50  0001 C CNN
+F 3 "" H 5500 4525 50  0001 C CNN
+	1    5500 4525
+	1    0    0    -1
+$EndComp
+Wire Wire Line
+	5500 3975 5500 3800
+Wire Wire Line
+	5500 3800 5850 3800
+Wire Wire Line
+	5500 4525 5500 4275
+Wire Wire Line
+	7600 2150 7600 2400
+Wire Wire Line
+	7700 2150 7700 2400
+$Comp
+L power:+5V #PWR0103
+U 1 1 5F2BFFED
+P 7700 2150
+F 0 "#PWR0103" H 7700 2000 50  0001 C CNN
+F 1 "+5V" V 7700 2400 50  0000 C CNN
+F 2 "" H 7700 2150 50  0001 C CNN
+F 3 "" H 7700 2150 50  0001 C CNN
+	1    7700 2150
+	1    0    0    -1
+$EndComp
+$Comp
+L power:+3V3 #PWR0102
+U 1 1 5F2BF89F
+P 7600 2150
+F 0 "#PWR0102" H 7600 2000 50  0001 C CNN
+F 1 "+3V3" V 7600 2400 50  0000 C CNN
+F 2 "" H 7600 2150 50  0001 C CNN
+F 3 "" H 7600 2150 50  0001 C CNN
+	1    7600 2150
+	1    0    0    -1
+$EndComp
