File: test/test.sch (KiCad schematic (older format))
At the start: 1 part

Commit message: more configs, runnig test, more putput
Parts:
- added C1: 100nF, Capacitor_SMD:C_1206_3216Metric, symbol Device:C
- added LOGO1: Logo_Open_Hardware_Large, Symbol:KiCad-Logo_5mm_SilkScreen, symbol Graphic:Logo_Open_Hardware_Large
- added R2: 100, Resistor_SMD:R_1206_3216Metric, symbol Device:R
- R1: footprint Resistor_THT:R_Axial_DIN0204_L3.6mm_D1.6mm_P7.62mm_Horizontal -> Resistor_SMD:R_1206_3216Metric; MPN (none) -> CRS1206-FX-1001ELF; Variant (none) -> +var1
Connections:
- net at R1.1, R1.2: now also C1.2
- new net: C1.1, R2.1, R2.2
Changed lines of the file:
@@
 Sheet 1 1
 Title "test"
-Date "2020-10-23"
-Rev "1"
+Date "2020-11-05"
+Rev "v1.1"
 Comp "nerdyscout"
 Comment1 ""
@@
 F 0 "R1" H 5100 3800 50  0000 L CNN
 F 1 "100" H 5100 3700 50  0000 L CNN
-F 2 "Resistor_THT:R_Axial_DIN0204_L3.6mm_D1.6mm_P7.62mm_Horizontal" V 4930 3725 50  0001 C CNN
+F 2 "Resistor_SMD:R_1206_3216Metric" V 4930 3725 50  0001 C CNN
 F 3 "~" H 5000 3725 50  0001 C CNN
+F 4 "+var1" H 5200 3625 50  0000 C CNN "Variant"
+F 5 "CRS1206-FX-1001ELF" H 5000 3725 50  0001 C CNN "MPN"
 	1    5000 3725
 	1    0    0    -1
@@
 Wire Wire Line
 	5000 3500 5000 3575
+$Comp
+L Device:R R2
+U 1 1 5FA43E0A
+P 6000 3725
+F 0 "R2" H 6100 3800 50  0000 L CNN
+F 1 "100" H 6100 3700 50  0000 L CNN
+F 2 "Resistor_SMD:R_1206_3216Metric" V 5930 3725 50  0001 C CNN
+F 3 "~" H 6000 3725 50  0001 C CNN
+F 4 "+var2" H 6175 3625 50  0000 C CNN "Variant"
+F 5 "CRS1206-FX-1001ELF" H 6000 3725 50  0001 C CNN "MPN"
+	1    6000 3725
+	1    0    0    -1
+$EndComp
+Wire Wire Line
+	6000 3875 6000 3925
+Wire Wire Line
+	6000 3925 5750 3925
+Wire Wire Line
+	5750 3925 5750 3500
+Wire Wire Line
+	5750 3500 6000 3500
+Wire Wire Line
+	6000 3500 6000 3575
+$Comp
+L Graphic:Logo_Open_Hardware_Large LOGO1
+U 1 1 5FA45422
+P 10500 5750
+F 0 "LOGO1" H 10500 6250 50  0001 C CNN
+F 1 "Logo_Open_Hardware_Large" H 10500 5350 50  0001 C CNN
+F 2 "Symbol:KiCad-Logo_5mm_SilkScreen" H 10500 5750 50  0001 C CNN
+F 3 "~" H 10500 5750 50  0001 C CNN
+	1    10500 5750
+	1    0    0    -1
+$EndComp
+$Comp
+L Device:C C1
+U 1 1 5FA45E53
+P 5375 3500
+F 0 "C1" V 5075 3525 50  0000 C CNN
+F 1 "100nF" V 5175 3525 50  0000 C CNN
+F 2 "Capacitor_SMD:C_1206_3216Metric" H 5413 3350 50  0001 C CNN
+F 3 "~" H 5375 3500 50  0001 C CNN
+F 4 "CL10B104JB8NNND" H 5375 3500 50  0001 C CNN "MPN"
+	1    5375 3500
+	0    1    1    0
+$EndComp
+Wire Wire Line
+	5225 3500 5000 3500
+Connection ~ 5000 3500
+Wire Wire Line
+	5525 3500 5750 3500
+Connection ~ 5750 3500
 $EndSCHEMATC
