File: test/test.sch (KiCad schematic (older format))
At the start: 5 parts

Commit message: changed test project
Parts:
- removed H1: MountingHole, MountingHole:MountingHole_2.7mm, symbol Mechanical:MountingHole
- added C2: 100nF, Capacitor_SMD:C_1206_3216Metric, symbol Device:C
- added U1: TLV70233_SOT23-5, Package_TO_SOT_SMD:SOT-23-5, symbol Regulator_Linear:TLV70233_SOT23-5
- added U2: FT230XQ, Package_DFN_QFN:QFN-16-1EP_4x4mm_P0.65mm_EP2.1x2.1mm, symbol Interface_USB:FT230XQ
- LOGO1: MPN (none) -> -
- R1: value 100 -> R; footprint Resistor_SMD:R_1206_3216Metric -> Resistor_SMD:R_0805_2012Metric; MPN CRS1206-FX-1001ELF -> (none); VARIANT (none) -> var1; Variant +var1 -> (none)
- R2: value 100 -> R; footprint Resistor_SMD:R_1206_3216Metric -> Resistor_SMD:R_0805_2012Metric; MPN CRS1206-FX-1001ELF -> 1; VARIANT (none) -> var2; Variant +var2 -> (none)
Connections:
- net GND: now reaches C1.2, R1.2
- net GND: now also R2.2, C2.1, U1.2 (GND), U2.13 (GND), U2.17 (GND), U2.3 (GND); no longer R1.1
- new net: C1.1, U1.1 (IN), U1.3 (EN)
- new net +3V3: C2.2, R1.1, R2.1, U1.5 (OUT), U2.1 (VCCIO), U2.10 (VCC)
- no-connect marks 0 -> 12
Other:
- moved on the sheet: C1
