File: test_data/test.kicad_pcb (KiCad board)
At the start: 2 copper layers, 20.3 x 20.3 mm, 5 parts, among them U1 TLV70233_SOT23-5, U2 FT230XQ

Commit message: moved kicad project used for test
Parts:
- added R1: R, Resistor_SMD:R_0805_2012Metric, F.Cu at (130.8, 92.1)
- added R2: R, Resistor_SMD:R_0805_2012Metric, F.Cu at (130.8, 97.2)
Routing:
- net +3V3: track 30.7 -> 33.4 mm
Changed lines of the file:
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@@
     (thickness 1.6)
     (drawings 7)
-    (tracks 23)
+    (tracks 28)
     (zones 0)
-    (modules 5)
+    (modules 7)
     (nets 4)
   )
@@
     (title test)
     (date 2020-10-23)
-    (rev v1)
+    (rev v2)
     (company nerdyscout)
   )
@@
     (add_net GND)
     (add_net "Net-(C1-Pad1)")
+  )
+  (module Resistor_SMD:R_0805_2012Metric (layer F.Cu)
+    (at 130.81 97.155)
+    (descr "Resistor SMD 0805 (2012 Metric), square (rectangular) end terminal, IPC_7351 nominal, (Body size source: https://docs.google.com/spreadsheets/d/1BsfQQcO9C6DZCsRaXUlFlo91Tg2WpOkGARC1WS5S8t0/edit?usp=sharing), generated with kicad-footprint-generator")
+    (tags resistor)
+    (attr smd)
+    (fp_text reference R2 (at 0 -1.65) (layer F.SilkS)
+      (effects (font (size 1 1) (thickness 0.15)))
+    )
+    (fp_text value R (at 0 1.65) (layer F.Fab)
+      (effects (font (size 1 1) (thickness 0.15)))
+    )
+    (fp_text user %R (at 0 0) (layer F.Fab)
+      (effects (font (size 0.5 0.5) (thickness 0.08)))
+    )
+    (fp_line (start 1.68 0.95) (end -1.68 0.95) (layer F.CrtYd) (width 0.05))
+    (fp_line (start 1.68 -0.95) (end 1.68 0.95) (layer F.CrtYd) (width 0.05))
+    (fp_line (start -1.68 -0.95) (end 1.68 -0.95) (layer F.CrtYd) (width 0.05))
+    (fp_line (start -1.68 0.95) (end -1.68 -0.95) (layer F.CrtYd) (width 0.05))
+    (fp_line (start -0.258578 0.71) (end 0.258578 0.71) (layer F.SilkS) (width 0.12))
+    (fp_line (start -0.258578 -0.71) (end 0.258578 -0.71) (layer F.SilkS) (width 0.12))
+    (fp_line (start 1 0.6) (end -1 0.6) (layer F.Fab) (width 0.1))
+    (fp_line (start 1 -0.6) (end 1 0.6) (layer F.Fab) (width 0.1))
+    (fp_line (start -1 -0.6) (end 1 -0.6) (layer F.Fab) (width 0.1))
+    (fp_line (start -1 0.6) (end -1 -0.6) (layer F.Fab) (width 0.1))
+    (pad 2 smd roundrect (at 0.9375 0) (size 0.975 1.4) (layers F.Cu F.Paste F.Mask) (roundrect_rratio 0.25)
+      (net 2 GND))
+    (pad 1 smd roundrect (at -0.9375 0) (size 0.975 1.4) (layers F.Cu F.Paste F.Mask) (roundrect_rratio 0.25)
+      (net 3 +3V3))
+    (model ${KISYS3DMOD}/Resistor_SMD.3dshapes/R_0805_2012Metric.wrl
+      (at (xyz 0 0 0))
+      (scale (xyz 1 1 1))
+      (rotate (xyz 0 0 0))
+    )
+  )
+  (module Resistor_SMD:R_0805_2012Metric (layer F.Cu)
+    (at 130.81 92.075)
+    (descr "Resistor SMD 0805 (2012 Metric), square (rectangular) end terminal, IPC_7351 nominal, (Body size source: https://docs.google.com/spreadsheets/d/1BsfQQcO9C6DZCsRaXUlFlo91Tg2WpOkGARC1WS5S8t0/edit?usp=sharing), generated with kicad-footprint-generator")
+    (tags resistor)
+    (attr smd)
+    (fp_text reference R1 (at 0 -1.65) (layer F.SilkS)
+      (effects (font (size 1 1) (thickness 0.15)))
+    )
+    (fp_text value R (at 0 1.65) (layer F.Fab)
+      (effects (font (size 1 1) (thickness 0.15)))
+    )
+    (fp_text user %R (at 0 0) (layer F.Fab)
+      (effects (font (size 0.5 0.5) (thickness 0.08)))
+    )
+    (fp_line (start 1.68 0.95) (end -1.68 0.95) (layer F.CrtYd) (width 0.05))
+    (fp_line (start 1.68 -0.95) (end 1.68 0.95) (layer F.CrtYd) (width 0.05))
+    (fp_line (start -1.68 -0.95) (end 1.68 -0.95) (layer F.CrtYd) (width 0.05))
+    (fp_line (start -1.68 0.95) (end -1.68 -0.95) (layer F.CrtYd) (width 0.05))
+    (fp_line (start -0.258578 0.71) (end 0.258578 0.71) (layer F.SilkS) (width 0.12))
+    (fp_line (start -0.258578 -0.71) (end 0.258578 -0.71) (layer F.SilkS) (width 0.12))
+    (fp_line (start 1 0.6) (end -1 0.6) (layer F.Fab) (width 0.1))
+    (fp_line (start 1 -0.6) (end 1 0.6) (layer F.Fab) (width 0.1))
+    (fp_line (start -1 -0.6) (end 1 -0.6) (layer F.Fab) (width 0.1))
+    (fp_line (start -1 0.6) (end -1 -0.6) (layer F.Fab) (width 0.1))
+    (pad 2 smd roundrect (at 0.9375 0) (size 0.975 1.4) (layers F.Cu F.Paste F.Mask) (roundrect_rratio 0.25)
+      (net 2 GND))
+    (pad 1 smd roundrect (at -0.9375 0) (size 0.975 1.4) (layers F.Cu F.Paste F.Mask) (roundrect_rratio 0.25)
+      (net 3 +3V3))
+    (model ${KISYS3DMOD}/Resistor_SMD.3dshapes/R_0805_2012Metric.wrl
+      (at (xyz 0 0 0))
+      (scale (xyz 1 1 1))
+      (rotate (xyz 0 0 0))
+    )
   )
   (module Package_DFN_QFN:QFN-16-1EP_4x4mm_P0.65mm_EP2.1x2.1mm (layer F.Cu)
@@
   (segment (start 132.395 103.825) (end 132.845 103.375) (width 0.25) (layer F.Cu) (net 3))
   (segment (start 126.41 96.21) (end 127.96 96.21) (width 0.25) (layer F.Cu) (net 3))
-  (segment (start 130.64 98.89) (end 130.64 103.825) (width 0.25) (layer F.Cu) (net 3))
-  (segment (start 127.96 96.21) (end 130.64 98.89) (width 0.25) (layer F.Cu) (net 3))
   (segment (start 127.96 91.765) (end 127.96 96.21) (width 0.25) (layer F.Cu) (net 3))
   (segment (start 127 90.805) (end 127.96 91.765) (width 0.25) (layer F.Cu) (net 3))
@@
   (segment (start 121.58 94.91) (end 121.285 94.615) (width 0.25) (layer F.Cu) (net 3))
   (segment (start 122.51 94.91) (end 121.58 94.91) (width 0.25) (layer F.Cu) (net 3))
+  (segment (start 128.905 97.155) (end 129.8725 97.155) (width 0.25) (layer F.Cu) (net 3))
+  (segment (start 127.96 96.21) (end 128.905 97.155) (width 0.25) (layer F.Cu) (net 3))
+  (segment (start 128.27 92.075) (end 127.96 91.765) (width 0.25) (layer F.Cu) (net 3))
+  (segment (start 129.8725 92.075) (end 128.27 92.075) (width 0.25) (layer F.Cu) (net 3))
+  (segment (start 129.8725 101.5725) (end 129.8725 97.155) (width 0.25) (layer F.Cu) (net 3))
+  (segment (start 130.64 102.34) (end 129.8725 101.5725) (width 0.25) (layer F.Cu) (net 3))
+  (segment (start 130.64 103.825) (end 130.64 102.34) (width 0.25) (layer F.Cu) (net 3))
   (zone (net 2) (net_name GND) (layer F.Cu) (hatch edge 0.508)
     (connect_pads (clearance 0.254))
